Commit message: feat: update IMU position to base_link center height in launch and URDF files

File: urdf/elderly_bot.urdf (robot description, URDF)
Before this commit: robot elderly_bot, 8 links, 7 joints
Joints:
- joint base_link_to_imu_link: origin xyz=0 0 0.05 rpy=0 0 0 -> xyz=0 0 0 rpy=0 0 0

Commit message: Add IMU mounting diagnostic and TF verification scripts
- Implemented imu_mounting_diagnostic.sh to determine IMU chip orientation relative to the robot's coordinate frame.
- Created tf_verification_complete.sh to verify laser rotation and diagnose IMU mounting orientation.
- Both scripts include detailed instructions, checks for prerequisites, and provide clear output for diagnostics.

File: urdf/elderly_bot.urdf (robot description, URDF)
Before this commit: robot elderly_bot, 8 links, 7 joints
Joints:
- joint base_link_to_laser: origin xyz=0 0 0.23 rpy=3.14159265359 0 0 -> xyz=0 0 0.23 rpy=0 0 3.14159265359

Commit message: fix: adjust IMU joint orientation for axis alignment with ROS REP-105

File: urdf/elderly_bot.urdf (robot description, URDF)
Before this commit: robot elderly_bot, 8 links, 7 joints
Joints:
- joint base_link_to_imu_link: origin xyz=0 0 0 rpy=0 0 0 -> xyz=0 0 0 rpy=0 0 3.14159265359

Commit message: fix: update WiFi credentials and server IP; adjust Madgwick filter parameters for improved stability; enhance master validation script for motor performance

File: urdf/elderly_bot.urdf (robot description, URDF)
Before this commit: robot elderly_bot, 8 links, 7 joints
Joints:
- joint base_link_to_imu_link: origin xyz=0 0 0 rpy=0 0 3.14159265359 -> xyz=0 0 0 rpy=3.14159265359 0 0

Commit message: fix: adjust Lidar mounting height and orientation for improved positioning

File: urdf/elderly_bot.urdf (robot description, URDF)
Before this commit: robot elderly_bot, 8 links, 7 joints
Joints:
- joint base_link_to_laser: origin xyz=0 0 0.23 rpy=0 0 3.14159265359 -> xyz=0 0 0.21 rpy=0 0 3.14159265359

Commit message: fix: update Lidar mounting description and correct IMU orientation for axis alignment

File: urdf/elderly_bot.urdf (robot description, URDF)
Before this commit: robot elderly_bot, 8 links, 7 joints
Joints:
- joint base_link_to_imu_link: origin xyz=0 0 0 rpy=3.14159265359 0 0 -> xyz=0 0 0 rpy=0 3.14159265359 0

Commit message: fix: correct IMU joint orientation for proper Z-axis alignment

File: urdf/elderly_bot.urdf (robot description, URDF)
Before this commit: robot elderly_bot, 8 links, 7 joints
Joints:
- joint base_link_to_imu_link: origin xyz=0 0 0 rpy=0 3.14159265359 0 -> xyz=0 0 0 rpy=3.14159265359 3.14159265359 0

Commit message: fix: adjust EKF yaw process noise covariance for improved IMU trust; update Madgwick filter zeta for stationary drift correction; modify URDF joint origin for better alignment

File: urdf/elderly_bot.urdf (robot description, URDF)
Before this commit: robot elderly_bot, 8 links, 7 joints
Joints:
- joint base_footprint_to_base_link: origin xyz=0 0 0.07 rpy=0 0 0 -> xyz=0 0 0.075 rpy=0 0 0

Commit message: fix: increase particle count for improved SLAM performance; adjust scan matching parameters for better accuracy

File: urdf/elderly_bot.urdf (robot description, URDF)
Before this commit: robot elderly_bot, 8 links, 7 joints
Joints:
- joint base_link_to_imu_link: origin xyz=0 0 0 rpy=3.14159265359 3.14159265359 0 -> xyz=0 0 0 rpy=0 3.14159265359 3.14159265359

Commit message: fix: correct IMU joint orientation for proper roll and pitch alignment

File: urdf/elderly_bot.urdf (robot description, URDF)
Before this commit: robot elderly_bot, 8 links, 7 joints
Joints:
- joint base_link_to_imu_link: origin xyz=0 0 0 rpy=0 3.14159265359 3.14159265359 -> xyz=0 0 0 rpy=3.14159265359 3.14159265359 0

Commit message: fix: update EKF process noise covariance for improved IMU trust; adjust GMapping scan matching parameters for better accuracy; modify URDF joint origins and wheel dimensions for correct alignment

File: urdf/elderly_bot.urdf (robot description, URDF)
Before this commit: robot elderly_bot, 8 links, 7 joints
Links:
- link front_left_wheel: geometry collision cylinder length=0.025 radius=0.0325; visual cylinder length=0.025 radius=0.0325
- link front_right_wheel: geometry collision cylinder length=0.025 radius=0.0325; visual cylinder length=0.025 radius=0.0325
- link rear_left_wheel: geometry collision cylinder length=0.025 radius=0.0325; visual cylinder length=0.025 radius=0.0325
- link rear_right_wheel: geometry collision cylinder length=0.025 radius=0.0325; visual cylinder length=0.025 radius=0.0325
Joints:
- joint base_footprint_to_base_link: origin xyz=0 0 0.075 rpy=0 0 0 -> xyz=0 0 0.0825 rpy=0 0 0
- joint base_link_to_imu_link: origin xyz=0 0 0 rpy=3.14159265359 3.14159265359 0 -> xyz=0 0 0 rpy=3.14159265359 0 0

Commit message: fix: adjust Madgwick filter zeta for optimal gyro bias drift correction; remap accelerometer and gyroscope data from NED to ROS ENU convention; correct IMU joint orientation in URDF for accurate alignment

File: urdf/elderly_bot.urdf (robot description, URDF)
Before this commit: robot elderly_bot, 8 links, 7 joints
Joints:
- joint base_link_to_imu_link: origin xyz=0 0 0 rpy=3.14159265359 0 0 -> xyz=0 0 0 rpy=0 0 0

Commit message: fix: disable linear acceleration in EKF configuration to prevent drift; update Lidar and IMU positions in URDF for accurate sensor alignment

File: urdf/elderly_bot.urdf (robot description, URDF)
Before this commit: robot elderly_bot, 8 links, 7 joints
Joints:
- joint base_link_to_imu_link: origin xyz=0 0 0 rpy=0 0 0 -> xyz=0 0 -0.0125 rpy=0 0 0
- joint base_link_to_laser: origin xyz=0 0 0.21 rpy=0 0 3.14159265359 -> xyz=0 0 0.14 rpy=0 0 3.14159265359

Commit message: Remove obsolete diagnostic scripts and update URDF for laser positioning
- Deleted the following scripts:
  - final_drift_validation.sh: Comprehensive validation of drift fixes.
  - imu_mounting_diagnostic.sh: Diagnostic for IMU physical mounting.
  - tf_verification_complete.sh: Complete TF verification for laser and IMU alignment.

- Updated the URDF file (elderly_bot.urdf) to adjust the laser's position relative to the IMU, changing the z-coordinate from 0.14m to 0.1275m to account for the IMU's height.

File: urdf/elderly_bot.urdf (robot description, URDF)
Before this commit: robot elderly_bot, 8 links, 7 joints
Joints:
- joint base_link_to_laser: origin xyz=0 0 0.14 rpy=0 0 3.14159265359 -> xyz=0 0 0.1275 rpy=0 0 3.14159265359

Commit message: feat: Update camera integration and setup script for AWS KVS compatibility

File: urdf/elderly_bot.urdf (robot description, URDF)
Before this commit: robot elderly_bot, 8 links, 7 joints
Links:
- added link camera_link, mass 0.05; visual box size=0.03 0.08 0.03
Joints:
- added joint base_link_to_camera_link: type fixed, parent base_link, child camera_link, origin xyz=0.15 0 0.25 rpy=0 0 0
